File: circuit/ACS758/voltage-sensor.sch (EAGLE design)
At the start: 6 parts, among them IC1 ACS758LCB-050B-PFF-T

Commit message: voltage and current sensor done
Parts:
- added R3: (no value), resistor:R-US_0207/10
- R1: device resistor:R-US_0207/10 -> resistor:R-US_M0805
Connections:
- removed net N$3: U$1.GND, U$2.GND
- new net GND_BAT: R3.1, U$1.GND, U$2.GND
- net GND: now also R3.2
Changed lines of the file:
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@@
 <part name="U$1" library="connector" deviceset="T-PLUG-FEMALE" device=""/>
 <part name="U$2" library="connector" deviceset="T-PLUG-MALE" device=""/>
-<part name="R1" library="resistor" deviceset="R-US_" device="0207/10"/>
+<part name="JP1" library="pinhead" deviceset="PINHD-1X4" device=""/>
+<part name="R1" library="resistor" deviceset="R-US_" device="M0805"/>
 <part name="R2" library="resistor" deviceset="R-US_" device="M0805"/>
-<part name="JP1" library="pinhead" deviceset="PINHD-1X4" device=""/>
+<part name="R3" library="resistor" deviceset="R-US_" device="0207/10"/>
 </parts>
 <sheets>
@@
 <instance part="U$1" gate="G$1" x="-2.54" y="45.72" rot="R180"/>
 <instance part="U$2" gate="G$1" x="53.34" y="45.72" rot="MR180"/>
+<instance part="JP1" gate="A" x="-20.32" y="22.86" rot="MR0"/>
 <instance part="R1" gate="G$1" x="43.18" y="30.48" rot="R90"/>
 <instance part="R2" gate="G$1" x="43.18" y="15.24" rot="R90"/>
-<instance part="JP1" gate="A" x="-20.32" y="22.86" rot="MR0"/>
+<instance part="R3" gate="G$1" x="43.18" y="2.54" rot="R90"/>
 </instances>
 <busses>
@@
 <nets>
 <net name="GND" class="0">
-<segment>
-<pinref part="R2" gate="G$1" pin="1"/>
-<wire x1="43.18" y1="10.16" x2="43.18" y2="5.08" width="0.1524" layer="91"/>
-<wire x1="43.18" y1="5.08" x2="50.8" y2="5.08" width="0.1524" layer="91"/>
-<label x="48.26" y="5.08" size="1.778" layer="95"/>
-</segment>
 <segment>
 <pinref part="IC1" gate="G$1" pin="GND"/>
@@
 <label x="-7.62" y="27.94" size="1.778" layer="95"/>
 </segment>
+<segment>
+<pinref part="R3" gate="G$1" pin="2"/>
+<pinref part="R2" gate="G$1" pin="1"/>
+<wire x1="43.18" y1="7.62" x2="43.18" y2="10.16" width="0.1524" layer="91"/>
+<wire x1="43.18" y1="7.62" x2="50.8" y2="7.62" width="0.1524" layer="91"/>
+<junction x="43.18" y="7.62"/>
+<label x="48.26" y="7.62" size="1.778" layer="95"/>
+</segment>
 </net>
 <net name="VBAT" class="0">
 <segment>
-<pinref part="R1" gate="G$1" pin="2"/>
 <wire x1="43.18" y1="35.56" x2="43.18" y2="43.18" width="0.1524" layer="91"/>
 <pinref part="U$2" gate="G$1" pin="VCC"/>
@@
 <wire x1="43.18" y1="43.18" x2="35.56" y2="43.18" width="0.1524" layer="91"/>
 <junction x="43.18" y="43.18"/>
+<pinref part="R1" gate="G$1" pin="2"/>
 </segment>
 </net>
 <net name="V_VOL" class="0">
 <segment>
-<pinref part="R1" gate="G$1" pin="1"/>
-<pinref part="R2" gate="G$1" pin="2"/>
 <wire x1="43.18" y1="25.4" x2="43.18" y2="22.86" width="0.1524" layer="91"/>
 <wire x1="43.18" y1="22.86" x2="43.18" y2="20.32" width="0.1524" layer="91"/>
@@
 <junction x="43.18" y="22.86"/>
 <label x="48.26" y="22.86" size="1.778" layer="95"/>
+<pinref part="R1" gate="G$1" pin="1"/>
+<pinref part="R2" gate="G$1" pin="2"/>
 </segment>
 <segment>
@@
 <wire x1="2.54" y1="43.18" x2="10.16" y2="43.18" width="0.1524" layer="91"/>
 <pinref part="IC1" gate="G$1" pin="IP-"/>
-</segment>
-</net>
-<net name="N$3" class="0">
-<segment>
-<pinref part="U$2" gate="G$1" pin="GND"/>
-<pinref part="U$1" gate="G$1" pin="GND"/>
-<wire x1="48.26" y1="48.26" x2="2.54" y2="48.26" width="0.1524" layer="91"/>
 </segment>
 </net>
@@
 </segment>
 </net>
+<net name="GND_BAT" class="0">
+<segment>
+<pinref part="U$2" gate="G$1" pin="GND"/>
+<pinref part="U$1" gate="G$1" pin="GND"/>
+<wire x1="48.26" y1="48.26" x2="15.24" y2="48.26" width="0.1524" layer="91"/>
+<wire x1="15.24" y1="48.26" x2="2.54" y2="48.26" width="0.1524" layer="91"/>
+<wire x1="15.24" y1="48.26" x2="15.24" y2="53.34" width="0.1524" layer="91"/>
+<junction x="15.24" y="48.26"/>
+<wire x1="15.24" y1="53.34" x2="20.32" y2="53.34" width="0.1524" layer="91"/>
+<label x="17.78" y="53.34" size="1.778" layer="95"/>
+</segment>
+<segment>
+<pinref part="R3" gate="G$1" pin="1"/>
+<wire x1="43.18" y1="-2.54" x2="43.18" y2="-5.08" width="0.1524" layer="91"/>
+<wire x1="43.18" y1="-5.08" x2="55.88" y2="-5.08" width="0.1524" layer="91"/>
+<label x="50.8" y="-5.08" size="1.778" layer="95"/>
+</segment>
+</net>

Commit message: layout done
Parts:
- added U$3: COOBOC, hqc-logo:COOBOC
Changed lines of the file:
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@@
 <layer number="97" name="Info" color="7" fill="1" visible="yes" active="yes"/>
 <layer number="98" name="Guide" color="6" fill="1" visible="yes" active="yes"/>
+<layer number="200" name="200bmp" color="1" fill="10" visible="yes" active="yes"/>
+<layer number="201" name="201bmp" color="2" fill="10" visible="yes" active="yes"/>
 </layers>
 <schematic xreflabel="%F%N/%S.%C%R" xrefpart="/%S.%C%R">
@@
 <part name="R2" library="resistor" deviceset="R-US_" device="M0805"/>
 <part name="R3" library="resistor" deviceset="R-US_" device="0207/10"/>
+<part name="U$3" library="hqc-logo" deviceset="COOBOC" device=""/>
 </parts>
 <sheets>
@@
 <instance part="R2" gate="G$1" x="43.18" y="15.24" rot="R90"/>
 <instance part="R3" gate="G$1" x="43.18" y="2.54" rot="R90"/>
+<instance part="U$3" gate="G$1" x="-10.16" y="10.16"/>
 </instances>
 <busses>

Commit message: add capicator on asc758
Parts:
- added C1: (no value), rcl:C-USC0805K
Connections:
- net GND: now also C1.2
- net VCC: now also C1.1
Changed lines of the file:
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@@
 <part name="R3" library="resistor" deviceset="R-US_" device="0207/10"/>
 <part name="U$3" library="hqc-logo" deviceset="COOBOC" device=""/>
+<part name="C1" library="rcl" deviceset="C-US" device="C0805K"/>
 </parts>
 <sheets>
@@
 <instance part="R3" gate="G$1" x="43.18" y="2.54" rot="R90"/>
 <instance part="U$3" gate="G$1" x="-10.16" y="10.16"/>
+<instance part="C1" gate="G$1" x="81.28" y="10.16"/>
 </instances>
 <busses>
@@
 <junction x="43.18" y="7.62"/>
 <label x="48.26" y="7.62" size="1.778" layer="95"/>
+</segment>
+<segment>
+<pinref part="C1" gate="G$1" pin="2"/>
+<wire x1="81.28" y1="5.08" x2="81.28" y2="2.54" width="0.1524" layer="91"/>
+<wire x1="81.28" y1="2.54" x2="86.36" y2="2.54" width="0.1524" layer="91"/>
+<label x="83.82" y="2.54" size="1.778" layer="95"/>
 </segment>
 </net>
@@
 <label x="-7.62" y="25.4" size="1.778" layer="95"/>
 </segment>
+<segment>
+<pinref part="C1" gate="G$1" pin="1"/>
+<wire x1="81.28" y1="12.7" x2="81.28" y2="15.24" width="0.1524" layer="91"/>
+<wire x1="81.28" y1="15.24" x2="86.36" y2="15.24" width="0.1524" layer="91"/>
+<label x="83.82" y="15.24" size="1.778" layer="95"/>
+</segment>
 </net>
