File: circuit/communication/crow.sch (EAGLE design)
At the start: 0 parts

Commit message: add modules on crow
Parts:
- added PCB1: ARDUINO_NANO, E14_Arduino_revB:ARDUINO_NANO
- added U$1, U$2: NRF24L01-AS01-ML01IPX, hqc-communication:NRF24L01-AS01-ML01IPX
- added U$3: 2.5W-TDD, hqc-communication:2.5W-TDD
Changed lines of the file:
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@@
 <grid distance="0.1" unitdist="inch" unit="inch" style="lines" multiple="1" display="no" altdistance="0.01" altunitdist="inch" altunit="inch"/>
 <layers>
+<layer number="1" name="Top" color="4" fill="1" visible="no" active="no"/>
+<layer number="16" name="Bottom" color="1" fill="1" visible="no" active="no"/>
+<layer number="17" name="Pads" color="2" fill="1" visible="no" active="no"/>
+<layer number="18" name="Vias" color="2" fill="1" visible="no" active="no"/>
+<layer number="19" name="Unrouted" color="6" fill="1" visible="no" active="no"/>
+<layer number="20" name="Dimension" color="15" fill="1" visible="no" active="no"/>
+<layer number="21" name="tPlace" color="7" fill="1" visible="no" active="no"/>
+<layer number="22" name="bPlace" color="7" fill="1" visible="no" active="no"/>
+<layer number="23" name="tOrigins" color="15" fill="1" visible="no" active="no"/>
+<layer number="24" name="bOrigins" color="15" fill="1" visible="no" active="no"/>
+<layer number="25" name="tNames" color="7" fill="1" visible="no" active="no"/>
+<layer number="26" name="bNames" color="7" fill="1" visible="no" active="no"/>
+<layer number="27" name="tValues" color="7" fill="1" visible="no" active="no"/>
+<layer number="28" name="bValues" color="7" fill="1" visible="no" active="no"/>
+<layer number="29" name="tStop" color="7" fill="3" visible="no" active="no"/>
+<layer number="30" name="bStop" color="7" fill="6" visible="no" active="no"/>
+<layer number="31" name="tCream" color="7" fill="4" visible="no" active="no"/>
+<layer number="32" name="bCream" color="7" fill="5" visible="no" active="no"/>
+<layer number="33" name="tFinish" color="6" fill="3" visible="no" active="no"/>
+<layer number="34" name="bFinish" color="6" fill="6" visible="no" active="no"/>
+<layer number="35" name="tGlue" color="7" fill="4" visible="no" active="no"/>
+<layer number="36" name="bGlue" color="7" fill="5" visible="no" active="no"/>
+<layer number="37" name="tTest" color="7" fill="1" visible="no" active="no"/>
+<layer number="38" name="bTest" color="7" fill="1" visible="no" active="no"/>
+<layer number="39" name="tKeepout" color="4" fill="11" visible="no" active="no"/>
+<layer number="40" name="bKeepout" color="1" fill="11" visible="no" active="no"/>
+<layer number="41" name="tRestrict" color="4" fill="10" visible="no" active="no"/>
+<layer number="42" name="bRestrict" color="1" fill="10" visible="no" active="no"/>
+<layer number="43" name="vRestrict" color="2" fill="10" visible="no" active="no"/>
+<layer number="44" name="Drills" color="7" fill="1" visible="no" active="no"/>
+<layer number="45" name="Holes" color="7" fill="1" visible="no" active="no"/>
+<layer number="46" name="Milling" color="3" fill="1" visible="no" active="no"/>
+<layer number="47" name="Measures" color="7" fill="1" visible="no" active="no"/>
+<layer number="48" name="Document" color="7" fill="1" visible="no" active="no"/>
+<layer number="49" name="Reference" color="7" fill="1" visible="no" active="no"/>
+<layer number="50" name="dxf" color="7" fill="1" visible="no" active="no"/>
+<layer number="51" name="tDocu" color="7" fill="1" visible="no" active="no"/>
+<layer number="52" name="bDocu" color="7" fill="1" visible="no" active="no"/>
+<layer number="53" name="tGND_GNDA" color="7" fill="9" visible="no" active="no"/>
+<layer number="54" name="bGND_GNDA" color="1" fill="9" visible="no" active="no"/>
+<layer number="56" name="wert" color="7" fill="1" visible="no" active="no"/>
 <layer number="90" name="Modules" color="5" fill="1" visible="yes" active="yes"/>
 <layer number="91" name="Nets" color="2" fill="1" visible="yes" active="yes"/>
@@
 <layer number="97" name="Info" color="7" fill="1" visible="yes" active="yes"/>
 <layer number="98" name="Guide" color="6" fill="1" visible="yes" active="yes"/>
+<layer number="100" name="Muster" color="7" fill="1" visible="no" active="no"/>
+<layer number="101" name="Patch_Top" color="12" fill="4" visible="yes" active="yes"/>
+<layer number="102" name="Vscore" color="7" fill="1" visible="yes" active="yes"/>
+<layer number="103" name="tMap" color="7" fill="1" visible="yes" active="yes"/>
+<layer number="104" name="Name" color="16" fill="1" visible="yes" active="yes"/>
+<layer number="105" name="tPlate" color="7" fill="1" visible="yes" active="yes"/>
+<layer number="106" name="bPlate" color="7" fill="1" visible="yes" active="yes"/>
+<layer number="107" name="Crop" color="7" fill="1" visible="yes" active="yes"/>
+<layer number="116" name="Patch_BOT" color="9" fill="4" visible="yes" active="yes"/>
+<layer number="121" name="_tsilk" color="7" fill="1" visible="yes" active="yes"/>
+<layer number="122" name="_bsilk" color="7" fill="1" visible="yes" active="yes"/>
+<layer number="125" name="_tNames" color="7" fill="1" visible="yes" active="yes"/>
+<layer number="144" name="Drill_legend" color="7" fill="1" visible="yes" active="yes"/>
+<layer number="151" name="HeatSink" color="7" fill="1" visible="yes" active="yes"/>
+<layer number="200" name="200bmp" color="1" fill="10" visible="yes" active="yes"/>
+<layer number="201" name="201bmp" color="2" fill="10" visible="yes" active="yes"/>
+<layer number="202" name="202bmp" color="3" fill="10" visible="yes" active="yes"/>
+<layer number="203" name="203bmp" color="4" fill="10" visible="yes" active="yes"/>
+<layer number="204" name="204bmp" color="5" fill="10" visible="yes" active="yes"/>
+<layer number="205" name="205bmp" color="6" fill="10" visible="yes" active="yes"/>
+<layer number="206" name="206bmp" color="7" fill="10" visible="yes" active="yes"/>
+<layer number="207" name="207bmp" color="8" fill="10" visible="yes" active="yes"/>
+<layer number="208" name="208bmp" color="9" fill="10" visible="yes" active="yes"/>
+<layer number="209" name="209bmp" color="7" fill="1" visible="yes" active="yes"/>
+<layer number="210" name="210bmp" color="7" fill="1" visible="yes" active="yes"/>
+<layer number="211" name="211bmp" color="7" fill="1" visible="yes" active="yes"/>
+<layer number="212" name="212bmp" color="7" fill="1" visible="yes" active="yes"/>
+<layer number="213" name="213bmp" color="7" fill="1" visible="yes" active="yes"/>
+<layer number="214" name="214bmp" color="7" fill="1" visible="yes" active="yes"/>
+<layer number="215" name="215bmp" color="7" fill="1" visible="yes" active="yes"/>
+<layer number="216" name="216bmp" color="7" fill="1" visible="yes" active="yes"/>
+<layer number="217" name="217bmp" color="18" fill="1" visible="no" active="no"/>
+<layer number="218" name="218bmp" color="19" fill="1" visible="no" active="no"/>
+<layer number="219" name="219bmp" color="20" fill="1" visible="no" active="no"/>
+<layer number="220" name="220bmp" color="21" fill="1" visible="no" active="no"/>
+<layer number="221" name="221bmp" color="22" fill="1" visible="no" active="no"/>
+<layer number="222" name="222bmp" color="23" fill="1" visible="no" active="no"/>
+<layer number="223" name="223bmp" color="24" fill="1" visible="no" active="no"/>
+<layer number="224" name="224bmp" color="25" fill="1" visible="no" active="no"/>
+<layer number="250" name="Descript" color="3" fill="1" visible="no" active="no"/>
+<layer number="251" name="SMDround" color="12" fill="11" visible="no" active="no"/>
+<layer number="254" name="cooling" color="7" fill="1" visible="yes" active="yes"/>
 </layers>
 <schematic xreflabel="%F%N/%S.%C%R" xrefpart="/%S.%C%R">
@@
 </classes>
 <parts>
+<part name="PCB1" library="E14_Arduino_revB" deviceset="ARDUINO_NANO" device=""/>
+<part name="U$1" library="hqc-communication" deviceset="NRF24L01-AS01-ML01IPX" device=""/>
+<part name="U$2" library="hqc-communication" deviceset="NRF24L01-AS01-ML01IPX" device=""/>
+<part name="U$3" library="hqc-communication" deviceset="2.5W-TDD" device=""/>
 </parts>
 <sheets>
@@
 </plain>
 <instances>
+<instance part="PCB1" gate="G$1" x="17.78" y="58.42" rot="R90"/>
+<instance part="U$1" gate="G$1" x="104.14" y="78.74"/>
+<instance part="U$2" gate="G$1" x="104.14" y="48.26"/>
+<instance part="U$3" gate="G$1" x="132.08" y="2.54"/>
 </instances>
 <busses>

Commit message: crow sch done
Parts:
- added C1: (no value), rcl:CPOL-USUD-5X5,8
- added JP1: (no value), pinhead:PINHD-1X2
- added JP2: M025MM, SparkFun-Connectors:M025MM
- added JP4: (no value), pinhead:PINHD-1X4
- added LED1: (no value), led:LEDSML0805
- added R1: 50, rcl:R-US_0207/10
- added R2, R3, R5, R6, R7, R8: 1k, rcl:R-US_0207/10
- added R4: 10k, rcl:R-US_0207/10
- added X1, X2: SMA-142-0701-801/806, con-coax:SMA-142-0701-801/806
- renumbered U$1 to RECV, U$2 to TRANSMITTER
Connections:
- new net 3V3: PCB1.3V3, RECV.3V3, TRANSMITTER.3V3
- new net 5V: C1.+, JP1.1, JP2.1, JP4.1, PCB1.5V, U$3.VPA
- new net D10: PCB1.D10, TRANSMITTER.CSN
- new net D2: PCB1.D2, R6.2
- new net D3: PCB1.D3, R7.2
- new net D5: PCB1.D5, R2.1, R4.1
- new net D6: PCB1.D6, R3.1, R5.1
- new net D7: PCB1.D7, RECV.CSN
- new net D8: PCB1.D8, RECV.CE
- new net D9: PCB1.D9, TRANSMITTER.CE
- new net GND: C1.-, JP1.2, JP2.2, JP4.4, PCB1.GND, PCB1.GND., R1.1, R4.2, R5.2, R8.2, RECV.GND, RECV.GND-ANT1, RECV.GND-ANT2, TRANSMITTER.GND, TRANSMITTER.GND-ANT1, TRANSMITTER.GND-ANT2, U$3.GND, U$3.GND-RX, U$3.GND-TX, U$3.GND1-ANT, U$3.GND2, U$3.GND2-ANT, U$3.GND3, U$3.GND4, U$3.GND5, U$3.GND6, U$3.RFIN, U$3.RFOUT, X1.2, X2.2
- new net MISO: PCB1.D12, RECV.MISO, TRANSMITTER.MISO
- new net MOSI: PCB1.D11, RECV.MOSI, TRANSMITTER.MOSI
- new net N$1: R1.2, U$3.GND-RFIN
- new net N$2: U$3.ANT, X1.1
- new net N$3: R7.1, TRANSMITTER.IRQ
- new net N$4: RECV.ANT, X2.1
- new net N$5: TRANSMITTER.ANT, U$3.GND-RFOUT
- new net N$6: R6.1, RECV.IRQ
- new net N$7: LED1.C, R8.1
- new net N$8: LED1.A, PCB1.D4
- new net RX: JP4.3, PCB1.RX0
- new net RXEN: R3.2, U$3.RX
- new net SCK: PCB1.D13, RECV.SCK, TRANSMITTER.SCK
- new net TX: JP4.2, PCB1.TX1
- new net TXEN: R2.2, U$3.TX
Other:
- moved on the sheet: U$3

Commit message: crow done, need print to check
Parts:
- PCB1: value ARDUINO_NANO -> ARDUINO_NANO_EXT; device E14_Arduino_revB:ARDUINO_NANO -> hqc-avr:ARDUINO_NANO_EXT
- R1, R2, R3, R4, R5, R6, R7, R8: device rcl:R-US_0207/10 -> rcl:R-US_M0805
Connections:
- net GND: now also LED1.C; no longer R8.2
- net N$7: now also PCB1.D4; no longer LED1.C
- net N$8: now also R8.2; no longer PCB1.D4
Other:
- moved on the sheet: LED1, R8
Changed lines of the file:
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@@
 <?xml version="1.0" encoding="utf-8"?>
 <!DOCTYPE eagle SYSTEM "eagle.dtd">
-<eagle version="7.0.0">
+<eagle version="7.2.0">
 <drawing>
 <settings>
@@
 <layers>
 <layer number="1" name="Top" color="4" fill="1" visible="yes" active="no"/>
+<layer number="2" name="Route2" color="1" fill="3" visible="yes" active="no"/>
+<layer number="3" name="Route3" color="4" fill="3" visible="yes" active="no"/>
+<layer number="4" name="Route4" color="1" fill="4" visible="yes" active="no"/>
+<layer number="5" name="Route5" color="4" fill="4" visible="yes" active="no"/>
+<layer number="6" name="Route6" color="1" fill="8" visible="yes" active="no"/>
+<layer number="7" name="Route7" color="4" fill="8" visible="yes" active="no"/>
+<layer number="8" name="Route8" color="1" fill="2" visible="yes" active="no"/>
+<layer number="9" name="Route9" color="4" fill="2" visible="yes" active="no"/>
+<layer number="10" name="Route10" color="1" fill="7" visible="yes" active="no"/>
+<layer number="11" name="Route11" color="4" fill="7" visible="yes" active="no"/>
+<layer number="12" name="Route12" color="1" fill="5" visible="yes" active="no"/>
+<layer number="13" name="Route13" color="4" fill="5" visible="yes" active="no"/>
+<layer number="14" name="Route14" color="1" fill="6" visible="yes" active="no"/>
+<layer number="15" name="Route15" color="4" fill="6" visible="yes" active="no"/>
 <layer number="16" name="Bottom" color="1" fill="1" visible="yes" active="no"/>
 <layer number="17" name="Pads" color="2" fill="1" visible="yes" active="no"/>
@@
 </classes>
 <parts>
-<part name="PCB1" library="E14_Arduino_revB" deviceset="ARDUINO_NANO" device=""/>
+<part name="PCB1" library="hqc-avr" deviceset="ARDUINO_NANO_EXT" device=""/>
 <part name="RECV" library="hqc-communication" deviceset="NRF24L01-AS01-ML01IPX" device=""/>
 <part name="TRANSMITTER" library="hqc-communication" deviceset="NRF24L01-AS01-ML01IPX" device=""/>
@@
 <part name="JP2" library="SparkFun-Connectors" deviceset="M02" device="5MM"/>
 <part name="SUPPLY5" library="supply2" deviceset="GND" device=""/>
-<part name="R1" library="rcl" deviceset="R-US_" device="0207/10" value="50"/>
+<part name="R1" library="rcl" deviceset="R-US_" device="M0805" value="50"/>
 <part name="SUPPLY6" library="supply2" deviceset="GND" device=""/>
 <part name="X1" library="con-coax" deviceset="SMA-" device="142-0701-801/806"/>
@@
 <part name="C1" library="rcl" deviceset="CPOL-US" device="UD-5X5,8"/>
 <part name="SUPPLY9" library="supply2" deviceset="GND" device=""/>
-<part name="R2" library="rcl" deviceset="R-US_" device="0207/10" value="1k"/>
-<part name="R3" library="rcl" deviceset="R-US_" device="0207/10" value="1k"/>
-<part name="R4" library="rcl" deviceset="R-US_" device="0207/10" value="10k"/>
-<part name="R5" library="rcl" deviceset="R-US_" device="0207/10" value="1k"/>
+<part name="R2" library="rcl" deviceset="R-US_" device="M0805" value="1k"/>
+<part name="R3" library="rcl" deviceset="R-US_" device="M0805" value="1k"/>
+<part name="R4" library="rcl" deviceset="R-US_" device="M0805" value="10k"/>
+<part name="R5" library="rcl" deviceset="R-US_" device="M0805" value="1k"/>
 <part name="SUPPLY10" library="supply2" deviceset="GND" device=""/>
 <part name="SUPPLY11" library="supply2" deviceset="GND" device=""/>
-<part name="R6" library="rcl" deviceset="R-US_" device="0207/10" value="1k"/>
-<part name="R7" library="rcl" deviceset="R-US_" device="0207/10" value="1k"/>
+<part name="R6" library="rcl" deviceset="R-US_" device="M0805" value="1k"/>
+<part name="R7" library="rcl" deviceset="R-US_" device="M0805" value="1k"/>
 <part name="JP4" library="pinhead" deviceset="PINHD-1X4" device=""/>
 <part name="LED1" library="led" deviceset="LED" device="SML0805"/>
-<part name="R8" library="rcl" deviceset="R-US_" device="0207/10" value="1k"/>
+<part name="R8" library="rcl" deviceset="R-US_" device="M0805" value="1k"/>
 <part name="SUPPLY12" library="supply2" deviceset="GND" device=""/>
 </parts>
@@
 <instance part="R7" gate="G$1" x="78.74" y="40.64" rot="R180"/>
 <instance part="JP4" gate="A" x="-104.14" y="66.04"/>
-<instance part="LED1" gate="G$1" x="-25.4" y="60.96" rot="R270"/>
-<instance part="R8" gate="G$1" x="-43.18" y="60.96" rot="R180"/>
+<instance part="LED1" gate="G$1" x="-33.02" y="60.96" rot="R270"/>
+<instance part="R8" gate="G$1" x="-20.32" y="60.96" rot="R180"/>
 <instance part="SUPPLY12" gate="GND" x="-50.8" y="55.88"/>
 </instances>
@@
 </segment>
 <segment>
+<pinref part="LED1" gate="G$1" pin="C"/>
 <pinref part="SUPPLY12" gate="GND" pin="GND"/>
-<wire x1="-50.8" y1="58.42" x2="-50.8" y2="60.96" width="0.1524" layer="91"/>
-<pinref part="R8" gate="G$1" pin="2"/>
-<wire x1="-50.8" y1="60.96" x2="-48.26" y2="60.96" width="0.1524" layer="91"/>
+<wire x1="-38.1" y1="60.96" x2="-50.8" y2="60.96" width="0.1524" layer="91"/>
+<wire x1="-50.8" y1="60.96" x2="-50.8" y2="58.42" width="0.1524" layer="91"/>
 </segment>
 </net>
@@
 <net name="N$7" class="0">
 <segment>
+<pinref part="PCB1" gate="G$1" pin="D4"/>
 <pinref part="R8" gate="G$1" pin="1"/>
-<pinref part="LED1" gate="G$1" pin="C"/>
-<wire x1="-38.1" y1="60.96" x2="-30.48" y2="60.96" width="0.1524" layer="91"/>
+<wire x1="2.54" y1="60.96" x2="-15.24" y2="60.96" width="0.1524" layer="91"/>
 </segment>
 </net>
 <net name="N$8" class="0">
 <segment>
+<pinref part="R8" gate="G$1" pin="2"/>
 <pinref part="LED1" gate="G$1" pin="A"/>
-<pinref part="PCB1" gate="G$1" pin="D4"/>
-<wire x1="-22.86" y1="60.96" x2="2.54" y2="60.96" width="0.1524" layer="91"/>
-</segment>
-</net>
+<wire x1="-25.4" y1="60.96" x2="-30.48" y2="60.96" width="0.1524" layer="91"/>
+</segment>
+</net>
